Commit message: Bug-fix: Changed the path to the robot meshes in the URDF

File: robot_model/mpo_500.urdf (robot description, URDF)
Before this commit: robot mmo_500, 8 links, 7 joints
Links:
- link base_footprint: geometry collision mesh filename=package://neo_mpo_500-2/robot_model/meshes/MPO_500/MPO-500-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 scale=0.001 0.001 0.001; visual mesh filename=package://neo_mpo_500-2/robot_model/meshes/MPO_500/MPO-500-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 scale=0.001 0.001 0.001
- link lidar_1_link: geometry collision mesh filename=package://neo_mpo_500-2/robot_model/meshes/MPO_500/SICK-S30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 scale=0.001 0.001 0.001; visual mesh filename=package://neo_mpo_500-2/robot_model/meshes/MPO_500/SICK-S30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 scale=0.001 0.001 0.001
- link lidar_2_link: geometry collision mesh filename=package://neo_mpo_500-2/robot_model/meshes/MPO_500/SICK-S30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 scale=0.001 0.001 0.001; visual mesh filename=package://neo_mpo_500-2/robot_model/meshes/MPO_500/SICK-S30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 scale=0.001 0.001 0.001
- link mpo_500_wheel_back_left_link: geometry collision mesh filename=package://neo_mpo_500-2/robot_model/meshes/MPO_500/MPO-500-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 scale=0.001 0.001 0.001; visual mesh filename=package://neo_mpo_500-2/robot_model/meshes/MPO_500/MPO-500-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 scale=0.001 0.001 0.001
- link mpo_500_wheel_back_right_link: geometry collision mesh filename=package://neo_mpo_500-2/robot_model/meshes/MPO_500/MPO-500-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 scale=0.001 0.001 0.001; visual mesh filename=package://neo_mpo_500-2/robot_model/meshes/MPO_500/MPO-500-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 scale=0.001 0.001 0.001
- link mpo_500_wheel_front_left_link: geometry collision mesh filename=package://neo_mpo_500-2/robot_model/meshes/MPO_500/MPO-500-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 scale=0.001 0.001 0.001; visual mesh filename=package://neo_mpo_500-2/robot_model/meshes/MPO_500/MPO-500-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 scale=0.001 0.001 0.001
- link mpo_500_wheel_front_right_link: geometry collision mesh filename=package://neo_mpo_500-2/robot_model/meshes/MPO_500/MPO-500-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 scale=0.001 0.001 0.001; visual mesh filename=package://neo_mpo_500-2/robot_model/meshes/MPO_500/MPO-500-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 scale=0.001 0.001 0.001
Joints:
- joint mpo_500_wheel_back_left_joint: type revolute -> fixed
- joint mpo_500_wheel_back_right_joint: type revolute -> fixed
- joint mpo_500_wheel_front_left_joint: type revolute -> fixed
- joint mpo_500_wheel_front_right_joint: type revolute -> fixed

Commit message: adding mmo_500 support

File: robot_model/mpo_500.urdf (robot description, URDF)
Before this commit: robot mmo_500, 8 links, 7 joints
Links:
- added link cabinet_link, mass 2; collision mesh filename=package://neo_mpo_500-2/robot_model/meshes/MPO_500/cabin.dae scale=0.001 0.001 0.001; visual mesh filename=package://neo_mpo_500-2/robot_model/meshes/MPO_500/cabin.dae scale=0.001 0.001 0.001
- added link ee_link; collision box size=0.01 0.01 0.01
- added link forearm_link, mass 3.87; collision mesh filename=package://neo_mpo_500-2/robot_model/meshes/ur10/visual/fore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; visual mesh filename=package://neo_mpo_500-2/robot_model/meshes/ur10/visual/fore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
- added link shoulder_link, mass 7.778; collision mesh filename=package://neo_mpo_500-2/robot_model/meshes/ur10/visual/shou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; visual mesh filename=package://neo_mpo_500-2/robot_model/meshes/ur10/visual/shou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
- added link upper_arm_link, mass 12.93; collision mesh filename=package://neo_mpo_500-2/robot_model/meshes/ur10/visual/uppe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; visual mesh filename=package://neo_mpo_500-2/robot_model/meshes/ur10/visual/uppe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
- added link ur10_base_link, mass 2.0; collision mesh filename=package://neo_mpo_500-2/robot_model/meshes/ur10/visual/base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; visual mesh filename=package://neo_mpo_500-2/robot_model/meshes/ur10/visual/base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
- added link wrist_1_link, mass 1.96; collision mesh filename=package://neo_mpo_500-2/robot_model/meshes/ur10/visual/wris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; visual mesh filename=package://neo_mpo_500-2/robot_model/meshes/ur10/visual/wris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
- added link wrist_2_link, mass 1.96; collision mesh filename=package://neo_mpo_500-2/robot_model/meshes/ur10/visual/wris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; visual mesh filename=package://neo_mpo_500-2/robot_model/meshes/ur10/visual/wris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
- added link wrist_3_link, mass 0.202; collision mesh filename=package://neo_mpo_500-2/robot_model/meshes/ur10/visual/wris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; visual mesh filename=package://neo_mpo_500-2/robot_model/meshes/ur10/visual/wris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
Joints:
- added joint cabinet_joint: type fixed, parent base_link, child cabinet_link, origin xyz=0.072 0 0.386 rpy=0 0 0
- added joint cabinet_u10_joint: type fixed, parent cabinet_link, child ur10_base_link, origin xyz=0.133 0.0 0.416 rpy=0.0 0.0 0.0
- added joint ee_fixed_joint: type fixed, parent wrist_3_link, child ee_link, origin xyz=0.0 0.0922 0.0 rpy=0.0 0.0 1.5707963267948966
- added joint elbow_joint: type revolute, parent upper_arm_link, child forearm_link, origin xyz=0.0 -0.1719 0.612 rpy=0.0 -1.95 0.0, axis 0 1 0, limit lower=-3.141592653589793 upper=3.141592653589793 effort=150.0 velocity=3.15
- added joint shoulder_lift_joint: type revolute, parent shoulder_link, child upper_arm_link, origin xyz=0.0 0.220941 0.0 rpy=0.0 -1.25 0.0, axis 0 1 0, limit lower=-3.141592653589793 upper=3.141592653589793 effort=330.0 velocity=2.16
- added joint shoulder_pan_joint: type revolute, parent ur10_base_link, child shoulder_link, origin xyz=0.0 0.0 0.1273 rpy=0.0 0.0 0.0, axis 0 0 1, limit lower=-3.141592653589793 upper=3.141592653589793 effort=330.0 velocity=2.16
- added joint wrist_1_joint: type revolute, parent forearm_link, child wrist_1_link, origin xyz=0.0 0.0 0.5723 rpy=0.0 1.5707963267948966 0.0, axis 0 1 0, limit lower=-3.141592653589793 upper=3.141592653589793 effort=54.0 velocity=3.2
- added joint wrist_2_joint: type revolute, parent wrist_1_link, child wrist_2_link, origin xyz=0.0 0.1149 0.0 rpy=0.0 0.0 0.0, axis 0 0 1, limit lower=-3.141592653589793 upper=3.141592653589793 effort=54.0 velocity=3.2
- added joint wrist_3_joint: type revolute, parent wrist_2_link, child wrist_3_link, origin xyz=0.0 0.0 0.1157 rpy=0.0 0.0 0.0, axis 0 1 0, limit lower=-3.141592653589793 upper=3.141592653589793 effort=54.0 velocity=3.2
