Commit message: Modified urdf to work with recent the changes in mesh name for cabinet in mp_components pkg

File: robot_model/mpo_500.urdf.xacro (robot description, xacro)
@@ -15,4 +15,5 @@
   <xacro:arg name="arm_parent" default="cabinet_link"/>
   <xacro:arg name="gripper_type" default=""/>
+  <xacro:arg name="use_ur_dc" default="false"/>
   <xacro:arg name="force_abs_paths" default="false"/>
   <xacro:arg name="simulation_controllers" default=""/>
@@ -29,4 +30,5 @@
   <xacro:property name="scanner_height" value="0"/>
   <xacro:property name="gripper" value="$(arg gripper_type)"/>
+  <xacro:property name="ur_dc" value="$(arg use_ur_dc)"/>
   <xacro:property name="use_mock" value="$(arg use_mock_hardware)"/>
   <!-- When there is an arm mounted, the joints of the wheels needs
@@ -104,8 +106,10 @@
     <!-- Universal Robotics (UR) Arms-->
     <xacro:if value="${arm == 'ur5' or arm == 'ur10' or arm == 'ur5e' or arm == 'ur10e'}">
+      <xacro:property name="arm_height" value="0.416" />
       <xacro:include filename="$(find mp_components)/urdf/arm/ur_arm.urdf.xacro"/>
     </xacro:if>
     <!-- Elite Arms-->
     <xacro:if value="${arm == 'ec66' or arm == 'cs66'}">
+      <xacro:property name="arm_height" value="0.376" />
       <xacro:include filename="$(find mp_components)/urdf/arm/elite_arm.urdf.xacro"/>
     </xacro:if>

Commit message: new hardware support

File: robot_model/mpo_500.urdf.xacro (robot description, xacro)
@@ -20,4 +20,5 @@
   <xacro:arg name="use_mock_hardware" default="false"/>
   <xacro:arg name="mock_sensor_commands" default="false"/>
+  <xacro:arg name="use_legacy" default="false"/>
   <xacro:arg name="include_arm_ros2_control" default="false"/>
   <xacro:arg name="include_gripper_ros2_control" default="false"/>
@@ -32,4 +33,5 @@
   <xacro:property name="ur_dc" value="$(arg use_ur_dc)"/>
   <xacro:property name="use_mock" value="$(arg use_mock_hardware)"/>
+  <xacro:property name="legacy" value="$(arg use_legacy)"/>
   <!-- When there is an arm mounted, the joints of the wheels needs
   to be of fixed type. The reason being, both the drive modules and
@@ -38,4 +40,10 @@
   to ROS 2 control. -->
   <xacro:property name="meca_joint_type" value="revolute"/>
+  <!-- Need to swap the model according to the legacy use -->
+  <xacro:property name="model" value="NEW"/>
+  <!-- use legacy -->
+  <xacro:if value="${legacy == True}">
+    <xacro:property name="model" value="LEGACY"/>
+  </xacro:if>
   <!-- Additionally for simulation, the joint type of the wheels needs to be fixed. -->
   <xacro:if value="${gz == True or use_mock == True}">
@@ -46,12 +54,18 @@
   <xacro:mpo_500_body/>
   <!-- Laser Scanners -->
-  <xacro:if value="${scanner == 'sick_s300'}">
-    <!--https://neobotix-docs.de/hardware/en/platforms/mpo-500/mechanical.html-->
-    <xacro:property name="scanner_height" value="0.372"/>
-    <xacro:include filename="$(find neo_mpo_500-2)/robot_model/xacros/sick_s300_macro.xacro"/>
+  <xacro:if value="${legacy == True}">
+    <xacro:if value="${scanner == 'sick_s300'}">
+      <!--https://neobotix-docs.de/hardware/en/platforms/mpo-500/mechanical.html-->
+      <xacro:property name="scanner_height" value="0.372"/>
+      <xacro:include filename="$(find neo_mpo_500-2)/robot_model/xacros/sick_s300_macro.xacro"/>
+    </xacro:if>
+    <xacro:if value="${scanner == 'sick_microscan3'}">
+      <xacro:property name="scanner_height" value="0.372"/>
+      <xacro:include filename="$(find neo_mpo_500-2)/robot_model/xacros/sick_microscan3_macro.xacro"/>
+    </xacro:if>
   </xacro:if>
-  <xacro:if value="${scanner == 'sick_microscan3'}">
-    <xacro:property name="scanner_height" value="0.372"/>
-    <xacro:include filename="$(find neo_mpo_500-2)/robot_model/xacros/sick_microscan3_macro.xacro"/>
+  <xacro:if value="${scanner == 'sick_nanoscan3'}">
+    <xacro:property name="scanner_height" value="0.386"/>
+    <xacro:include filename="$(find neo_mpo_500-2)/robot_model/xacros/sick_nanoscan.xacro"/>
   </xacro:if>
   <xacro:sick_laser_scanner

File: robot_model/xacros/mpo_500_body.urdf.xacro (robot description, xacro)
@@ -25,5 +25,5 @@
           <origin rpy="-1.571 0 1.571" xyz="0 0 0"/>
           <geometry>
-            <mesh filename="package://neo_mpo_500-2/robot_model/meshes/MPO-500-BODY.dae" scale="0.001 0.001 0.001"/>
+            <mesh filename="package://neo_mpo_500-2/robot_model/meshes/MPO-500-BODY-${model}.dae" scale="0.001 0.001 0.001"/>
           </geometry>
         </visual>
@@ -31,5 +31,5 @@
           <origin rpy="-1.571 0 1.571" xyz="0 0 0"/>
           <geometry>
-            <mesh filename="package://neo_mpo_500-2/robot_model/meshes/MPO-500-BODY.dae" scale="0.001 0.001 0.001"/>
+            <mesh filename="package://neo_mpo_500-2/robot_model/meshes/MPO-500-BODY-${model}.dae" scale="0.001 0.001 0.001"/>
           </geometry>
         </collision>

Commit message: new hardware update

File: robot_model/mpo_500.urdf.xacro (robot description, xacro)
@@ -19,4 +19,5 @@
   <xacro:arg name="use_mock_hardware" default="false"/>
   <xacro:arg name="mock_sensor_commands" default="false"/>
+  <xacro:arg name="use_legacy" default="false"/>
   <xacro:arg name="include_arm_ros2_control" default="false"/>
   <xacro:arg name="include_gripper_ros2_control" default="false"/>
@@ -30,4 +31,5 @@
   <xacro:property name="ur_dc" value="$(arg use_ur_dc)"/>
   <xacro:property name="use_mock" value="$(arg use_mock_hardware)"/>
+  <xacro:property name="legacy" value="$(arg use_legacy)"/>
   <!-- When there is an arm mounted, the joints of the wheels needs
   to be of fixed type. The reason being, both the drive modules and
@@ -36,16 +38,28 @@
   to ROS 2 control. -->
   <xacro:property name="meca_joint_type" value="revolute"/>
+  <!-- Need to swap the model according to the legacy use -->
+  <xacro:property name="model" value="NEW"/>
+  <!-- use legacy -->
+  <xacro:if value="${legacy == True}">
+    <xacro:property name="model" value="LEGACY"/>
+  </xacro:if>
   <!-- Include the robot body -->
   <xacro:include filename="$(find neo_mpo_500-2)/robot_model/xacros/mpo_500_body.urdf.xacro"/>
   <xacro:mpo_500_body/>
   <!-- Laser Scanners -->
-  <xacro:if value="${scanner == 'sick_s300'}">
-    <!--https://neobotix-docs.de/hardware/en/platforms/mpo-500/mechanical.html-->
-    <xacro:property name="scanner_height" value="0.372"/>
-    <xacro:include filename="$(find neo_mpo_500-2)/robot_model/xacros/sick_s300_macro.xacro"/>
+  <xacro:if value="${legacy == True}">
+    <xacro:if value="${scanner == 'sick_s300'}">
+      <!--https://neobotix-docs.de/hardware/en/platforms/mpo-500/mechanical.html-->
+      <xacro:property name="scanner_height" value="0.372"/>
+      <xacro:include filename="$(find neo_mpo_500-2)/robot_model/xacros/sick_s300_macro.xacro"/>
+    </xacro:if>
+    <xacro:if value="${scanner == 'sick_microscan3'}">
+      <xacro:property name="scanner_height" value="0.372"/>
+      <xacro:include filename="$(find neo_mpo_500-2)/robot_model/xacros/sick_microscan3_macro.xacro"/>
+    </xacro:if>
   </xacro:if>
-  <xacro:if value="${scanner == 'sick_microscan3'}">
-    <xacro:property name="scanner_height" value="0.372"/>
-    <xacro:include filename="$(find neo_mpo_500-2)/robot_model/xacros/sick_microscan3_macro.xacro"/>
+  <xacro:if value="${scanner == 'sick_nanoscan3'}">
+    <xacro:property name="scanner_height" value="0.386"/>
+    <xacro:include filename="$(find neo_mpo_500-2)/robot_model/xacros/sick_nanoscan.xacro"/>
   </xacro:if>
   <xacro:sick_laser_scanner

Commit message: updates for new hardware

File: robot_model/mpo_500.urdf.xacro (robot description, xacro)
@@ -7,5 +7,4 @@
 <!-- This is the main URDF file for mpo_700-->
   <!-- Xacro Arguments-->
-  <xacro:arg name="use_gz" default="false"/>
   <xacro:arg name="use_imu" default="false"/>
   <xacro:arg name="use_d435" default="false"/>
@@ -24,5 +23,4 @@
   <!-- Xacro Properties -->
   <xacro:property name="arm" value="$(arg arm_type)"/>
-  <xacro:property name="gz" value="$(arg use_gz)"/>
   <xacro:property name="imu" value="$(arg use_imu)"/>
   <xacro:property name="d435" value="$(arg use_d435)"/>
@@ -38,8 +36,4 @@
   to ROS 2 control. -->
   <xacro:property name="meca_joint_type" value="revolute"/>
-  <!-- Additionally for simulation, the joint type of the wheels needs to be fixed. -->
-  <xacro:if value="${gz == True or arm != ''}">
-    <xacro:property name="meca_joint_type" value="fixed"/>
-  </xacro:if>
   <!-- Include the robot body -->
   <xacro:include filename="$(find neo_mpo_500-2)/robot_model/xacros/mpo_500_body.urdf.xacro"/>
@@ -131,5 +125,4 @@
           use_mock_hardware="${use_mock}"
           mock_sensor_commands="${use_mock}"
-          sim_gazebo="${gz}"
           include_ros2_control="$(arg include_gripper_ros2_control)"
           >
@@ -147,8 +140,3 @@
     </xacro:unless>
   </xacro:unless>
-  <!-- Simulation -->
-  <xacro:if value="${gz == True}">
-    <xacro:include filename="$(find mp_components)/urdf/gazebo/mpo_500/mpo_500_gazebo.urdf.xacro" />
-    <xacro:mpo_500_gazebo />
-  </xacro:if>
 </robot>

Commit message: updates for scanner dimension

File: robot_model/mpo_500.urdf.xacro (robot description, xacro)
@@ -51,14 +51,14 @@
     <xacro:if value="${scanner == 'sick_s300'}">
       <!--https://neobotix-docs.de/hardware/en/platforms/mpo-500/mechanical.html-->
-      <xacro:property name="scanner_height" value="0.372"/>
+      <xacro:property name="scanner_x_value" value="0.442"/>
       <xacro:include filename="$(find neo_mpo_500-2)/robot_model/xacros/sick_s300_macro.xacro"/>
     </xacro:if>
     <xacro:if value="${scanner == 'sick_microscan3'}">
-      <xacro:property name="scanner_height" value="0.372"/>
+      <xacro:property name="scanner_x_value" value="0.442"/>
       <xacro:include filename="$(find neo_mpo_500-2)/robot_model/xacros/sick_microscan3_macro.xacro"/>
     </xacro:if>
   </xacro:if>
   <xacro:if value="${scanner == 'sick_nanoscan3'}">
-    <xacro:property name="scanner_height" value="0.386"/>
+    <xacro:property name="scanner_x_value" value="0.454"/>
     <xacro:include filename="$(find neo_mpo_500-2)/robot_model/xacros/sick_nanoscan.xacro"/>
   </xacro:if>
@@ -67,5 +67,5 @@
     parent="base_link"
     >
-    <origin rpy="0 0 0" xyz="0.442 0 ${scanner_height}"/>
+    <origin rpy="0 0 0" xyz="${scanner_x_value} 0 0.372"/>
   </xacro:sick_laser_scanner>
   <xacro:sick_laser_scanner
@@ -73,5 +73,5 @@
     parent="base_link"
     >
-    <origin rpy="0 0 3.14" xyz="-0.442 0 ${scanner_height}"/>
+    <origin rpy="0 0 3.14" xyz="-${scanner_x_value} 0 0.372"/>
   </xacro:sick_laser_scanner>
   <!-- Using IMU -->

Commit message: updates for scanner dimension

File: robot_model/mpo_500.urdf.xacro (robot description, xacro)
@@ -57,14 +57,14 @@
     <xacro:if value="${scanner == 'sick_s300'}">
       <!--https://neobotix-docs.de/hardware/en/platforms/mpo-500/mechanical.html-->
-      <xacro:property name="scanner_height" value="0.372"/>
+      <xacro:property name="scanner_x_value" value="0.442"/>
       <xacro:include filename="$(find neo_mpo_500-2)/robot_model/xacros/sick_s300_macro.xacro"/>
     </xacro:if>
     <xacro:if value="${scanner == 'sick_microscan3'}">
-      <xacro:property name="scanner_height" value="0.372"/>
+      <xacro:property name="scanner_x_value" value="0.442"/>
       <xacro:include filename="$(find neo_mpo_500-2)/robot_model/xacros/sick_microscan3_macro.xacro"/>
     </xacro:if>
   </xacro:if>
   <xacro:if value="${scanner == 'sick_nanoscan3'}">
-    <xacro:property name="scanner_height" value="0.386"/>
+    <xacro:property name="scanner_x_value" value="0.454"/>
     <xacro:include filename="$(find neo_mpo_500-2)/robot_model/xacros/sick_nanoscan.xacro"/>
   </xacro:if>
@@ -73,5 +73,5 @@
     parent="base_link"
     >
-    <origin rpy="0 0 0" xyz="0.442 0 ${scanner_height}"/>
+    <origin rpy="0 0 0" xyz="${scanner_x_value} 0 0.372"/>
   </xacro:sick_laser_scanner>
   <xacro:sick_laser_scanner
@@ -79,5 +79,5 @@
     parent="base_link"
     >
-    <origin rpy="0 0 3.14" xyz="-0.442 0 ${scanner_height}"/>
+    <origin rpy="0 0 3.14" xyz="-${scanner_x_value} 0 0.372"/>
   </xacro:sick_laser_scanner>
   <!-- Using IMU -->
