Commit message: update robot model, launch and add UR support

File: robot_model/mpo_500/mpo_500.urdf.xacro (robot description, xacro)
@@ -1,18 +1,22 @@
-<?xml version="1.0" encoding="utf-8"?>
-<!-- =================================================================================== -->
-<!-- |    This document was autogenerated by xacro from mpo_500.urdf.xacro             | -->
-<!-- |    EDITING THIS FILE BY HAND IS NOT RECOMMENDED                                 | -->
-<!-- =================================================================================== -->
-<robot name="mmo_500">
-  <!-- Microscan - Comment/Uncomment if required -->
-  <!-- <xacro:include filename="$(find neo_mpo_500-2)/robot_model/urdf/mpo_500_xacros/micro_scan.xacro" />-->
-  <!-- USS and IMU - Comment/Uncomment if required  -->
-  <!--<xacro:include filename="$(find neo_mpo_500-2)/robot_model/urdf/mpo_500_xacros/imu.xacro" />
-    <xacro:include filename="$(find neo_mpo_500-2)/robot_model/mmo_500/urdf/mpo_500_xacros/ultrasonic.xacro" /> -->
-  <!--ur10 -->
-  <!-- <xacro:include filename="$(find neo_mpo_500-2)/robot_model/urdf/ur10.urdf.xacro" /> -->
-  <!-- Base Macro-->
+<?xml version="1.0" ?>
+<robot xmlns:xacro="http://www.ros.org/wiki/xacro" name="mpo_700">
+  <!-- SENSORS -->
+  <xacro:arg name="arm_type" default=""/>
+  <xacro:arg name="use_imu" default="false"/>
+  <xacro:arg name="use_d435" default="false"/>
+  <xacro:property name="arm" value="$(arg arm_type)"/>
+  <xacro:property name="imu" value="$(arg use_imu)"/>
+  <xacro:property name="d435" value="$(arg use_d435)"/>
+  <!-- When there is an arm mounted, the joints of the wheels needs
+  to be of fixed type. The reason being, both the drive modules and
+  the arm cannot publish joint states simultenously. Thus we omit
+  the visualization of the drives. Issue will be fixed, when we switch
+  to ROS 2 control. -->
+  <xacro:property name="meca_joint_type" value="revolute"/>
+  <xacro:unless value="${arm == ''}">
+    <xacro:property name="meca_joint_type" value="fixed"/>
+  </xacro:unless>
   <link name="base_link"/>
-  <joint name="base_footprint_joint" type="fixed">
+  <joint name="base_footprint_joint" type="${meca_joint_type}">
     <origin rpy="0 0 0" xyz="0 0 0"/>
     <axis xyz="0 0 -1"/>
@@ -21,5 +25,4 @@
     <child link="base_footprint"/>
   </joint>
-  <!-- Link -->
   <link name="base_footprint">
     <inertial>
@@ -37,10 +40,9 @@
       <origin rpy="-1.571 0 1.571" xyz="0. 0. 0.0"/>
       <geometry>
-        <!--<box size="0.68 0.41 0.25"/> -->
         <mesh filename="package://neo_mpo_500-2/robot_model/meshes/MPO_500/MPO-500-BODY.dae" scale="0.001 0.001 0.001"/>
       </geometry>
     </collision>
   </link>
-  <joint name="mpo_500_wheel_front_left_joint" type="fixed">
+  <joint name="wheel_front_left_joint" type="${meca_joint_type}">
     <origin rpy="0 0 0" xyz="0.25 0.28 0.13"/>
     <axis xyz="0 1 0"/>
@@ -49,26 +51,26 @@
     <joint_properties damping="1.0" friction="1"/>
     <parent link="base_footprint"/>
-    <child link="mpo_500_wheel_front_left_link"/>
-  </joint>
-  <link name="mpo_500_wheel_front_left_link" type="wheel">
-    <inertial>
-      <mass value="1"/>
-      <origin rpy="0 0 0" xyz="0 0 0"/>
-      <inertia ixx="0.00044332" ixy="0" ixz="0" iyy="0.00044332" iyz="0" izz="0.00072"/>
-    </inertial>
-    <visual>
-      <origin rpy="0 0 0" xyz="0 0 0"/>
-      <geometry>
-        <mesh filename="package://neo_mpo_500-2/robot_model/meshes/MPO_500/MPO-500-WHEEL.dae" scale="0.001 0.001 0.001"/>
-      </geometry>
-    </visual>
-    <collision>
-      <origin rpy="0 0 0" xyz="0 0 0"/>
-      <geometry>
-        <mesh filename="package://neo_mpo_500-2/robot_model/meshes/MPO_500/MPO-500-WHEEL.dae" scale="0.001 0.001 0.001"/>
-      </geometry>
-    </collision>
-  </link>
-  <joint name="mpo_500_wheel_front_right_joint" type="fixed">
+    <child link="wheel_front_left_link"/>
+  </joint>
+  <link name="wheel_front_left_link">
+    <inertial>
+      <mass value="1"/>
+      <origin rpy="0 0 0" xyz="0 0 0"/>
+      <inertia ixx="0.00044332" ixy="0" ixz="0" iyy="0.00044332" iyz="0" izz="0.00072"/>
+    </inertial>
+    <visual>
+      <origin rpy="0 0 0" xyz="0 0 0"/>
+      <geometry>
+        <mesh filename="package://neo_mpo_500-2/robot_model/meshes/MPO_500/MPO-500-WHEEL.dae" scale="0.001 0.001 0.001"/>
+      </geometry>
+    </visual>
+    <collision>
+      <origin rpy="0 0 0" xyz="0 0 0"/>
+      <geometry>
+        <mesh filename="package://neo_mpo_500-2/robot_model/meshes/MPO_500/MPO-500-WHEEL.dae" scale="0.001 0.001 0.001"/>
+      </geometry>
+    </collision>
+  </link>
+  <joint name="wheel_front_right_joint" type="${meca_joint_type}">
     <origin rpy="0 0 3.14" xyz="0.25 -0.28 0.13"/>
     <axis xyz="0 1 0"/>
@@ -77,26 +79,26 @@
     <joint_properties damping="1.0" friction="1"/>
     <parent link="base_footprint"/>
-    <child link="mpo_500_wheel_front_right_link"/>
-  </joint>
-  <link name="mpo_500_wheel_front_right_link" type="wheel">
-    <inertial>
-      <mass value="1"/>
-      <origin rpy="0 0 0" xyz="0 0 0"/>
-      <inertia ixx="0.00044332" ixy="0" ixz="0" iyy="0.00044332" iyz="0" izz="0.00072"/>
-    </inertial>
-    <visual>
-      <origin rpy="0 0 0" xyz="0 0 0"/>
-      <geometry>
-        <mesh filename="package://neo_mpo_500-2/robot_model/meshes/MPO_500/MPO-500-WHEEL.dae" scale="0.001 0.001 0.001"/>
-      </geometry>
-    </visual>
-    <collision>
-      <origin rpy="0 0 0" xyz="0 0 0"/>
-      <geometry>
-        <mesh filename="package://neo_mpo_500-2/robot_model/meshes/MPO_500/MPO-500-WHEEL.dae" scale="0.001 0.001 0.001"/>
-      </geometry>
-    </collision>
-  </link>
-  <joint name="mpo_500_wheel_back_left_joint" type="fixed">
+    <child link="wheel_front_right_link"/>
+  </joint>
+  <link name="wheel_front_right_link">
+    <inertial>
+      <mass value="1"/>
+      <origin rpy="0 0 0" xyz="0 0 0"/>
+      <inertia ixx="0.00044332" ixy="0" ixz="0" iyy="0.00044332" iyz="0" izz="0.00072"/>
+    </inertial>
+    <visual>
+      <origin rpy="0 0 0" xyz="0 0 0"/>
+      <geometry>
+        <mesh filename="package://neo_mpo_500-2/robot_model/meshes/MPO_500/MPO-500-WHEEL.dae" scale="0.001 0.001 0.001"/>
+      </geometry>
+    </visual>
+    <collision>
+      <origin rpy="0 0 0" xyz="0 0 0"/>
+      <geometry>
+        <mesh filename="package://neo_mpo_500-2/robot_model/meshes/MPO_500/MPO-500-WHEEL.dae" scale="0.001 0.001 0.001"/>
+      </geometry>
+    </collision>
+  </link>
+  <joint name="wheel_back_left_joint" type="${meca_joint_type}">
     <origin rpy="0 0 0" xyz="-0.25 0.28 0.13"/>
     <axis xyz="0 1 0"/>
@@ -105,26 +107,26 @@
     <joint_properties damping="1.0" friction="1"/>
     <parent link="base_footprint"/>
-    <child link="mpo_500_wheel_back_left_link"/>
-  </joint>
-  <link name="mpo_500_wheel_back_left_link" type="wheel">
-    <inertial>
-      <mass value="1"/>
-      <origin rpy="0 0 0" xyz="0 0 0"/>
-      <inertia ixx="0.00044332" ixy="0" ixz="0" iyy="0.00044332" iyz="0" izz="0.00072"/>
-    </inertial>
-    <visual>
-      <origin rpy="0 0 0" xyz="0 0 0"/>
-      <geometry>
-        <mesh filename="package://neo_mpo_500-2/robot_model/meshes/MPO_500/MPO-500-WHEEL.dae" scale="0.001 0.001 0.001"/>
-      </geometry>
-    </visual>
-    <collision>
-      <origin rpy="0 0 0" xyz="0 0 0"/>
-      <geometry>
-        <mesh filename="package://neo_mpo_500-2/robot_model/meshes/MPO_500/MPO-500-WHEEL.dae" scale="0.001 0.001 0.001"/>
-      </geometry>
-    </collision>
-  </link>
-  <joint name="mpo_500_wheel_back_right_joint" type="fixed">
+    <child link="wheel_back_left_link"/>
+  </joint>
+  <link name="wheel_back_left_link">
+    <inertial>
+      <mass value="1"/>
+      <origin rpy="0 0 0" xyz="0 0 0"/>
+      <inertia ixx="0.00044332" ixy="0" ixz="0" iyy="0.00044332" iyz="0" izz="0.00072"/>
+    </inertial>
+    <visual>
+      <origin rpy="0 0 0" xyz="0 0 0"/>
+      <geometry>
+        <mesh filename="package://neo_mpo_500-2/robot_model/meshes/MPO_500/MPO-500-WHEEL.dae" scale="0.001 0.001 0.001"/>
+      </geometry>
+    </visual>
+    <collision>
+      <origin rpy="0 0 0" xyz="0 0 0"/>
+      <geometry>
+        <mesh filename="package://neo_mpo_500-2/robot_model/meshes/MPO_500/MPO-500-WHEEL.dae" scale="0.001 0.001 0.001"/>
+      </geometry>
+    </collision>
+  </link>
+  <joint name="wheel_back_right_joint" type="${meca_joint_type}">
     <origin rpy="0 0 3.14" xyz="-0.25 -0.28 0.13"/>
     <axis xyz="0 1 0"/>
@@ -133,7 +135,7 @@
     <joint_properties damping="1.0" friction="1"/>
     <parent link="base_footprint"/>
-    <child link="mpo_500_wheel_back_right_link"/>
-  </joint>
-  <link name="mpo_500_wheel_back_right_link" type="wheel">
+    <child link="wheel_back_right_link"/>
+  </joint>
+  <link name="wheel_back_right_link">
     <inertial>
       <mass value="1"/>
@@ -160,5 +162,5 @@
     <child link="lidar_1_link"/>
   </joint>
-  <link name="lidar_1_link" type="laser">
+  <link name="lidar_1_link">
     <inertial>
       <mass value="0.001"/>
@@ -185,5 +187,5 @@
     <child link="lidar_2_link"/>
   </joint>
-  <link name="lidar_2_link" type="laser">
+  <link name="lidar_2_link">
     <inertial>
       <mass value="0.001"/>
@@ -204,105 +206,81 @@
     </collision>
   </link>
-  <!--+++++++++++++++++++ IMU ++++++++++++++++++++++++-->
-  <!-- Comment or uncomment based on your requirement -->
-  <!--   <xacro:imu name="imu_1" parent="base_link">
-    <origin xyz="0.100 0 0.300" rpy="0 0 3.14" />
-  </xacro:imu> -->
-  <!--+++++++++++++++++++ Ultra Sonic ++++++++++++++++++++++++-->
-  <!-- Comment or uncomment based on your requirement -->
-  <!-- SENSOR 1 -->
-  <!-- xacro:us_sensor name="us_1" parent="base_link">
-    <origin xyz="0.100 0 0.300" rpy="0 3.14 3.14" />
-  </xacro:us_sensor-->
-  <!-- SENSOR 2 -->
-  <!-- xacro:us_sensor name="us_2" parent="base_link">
-    <origin xyz="0.110 0 0.300" rpy="0 3.14 3.14" />
-  </xacro:us_sensor-->
-  <!-- SENSOR 3 -->
-  <!-- xacro:us_sensor name="us_3" parent="base_link">
-    <origin xyz="0.120 0 0.300" rpy="0 3.14 3.14" />
-  </xacro:us_sensor-->
-  <!-- SENSOR 4 -->
-  <!-- xacro:us_sensor name="us_4" parent="base_link">
-    <origin xyz="0.130 0 0.300" rpy="0 3.14 3.14" />
-  </xacro:us_sensor-->
-  <!-- SENSOR 5 -->
-  <!-- xacro:us_sensor name="us_5" parent="base_link">
-    <origin xyz="0.140 0 0.300" rpy="0 3.14 3.14" />
-  </xacro:us_sensor-->
-  <!-- SENSOR 6 -->
-  <!-- xacro:us_sensor name="us_6" parent="base_link">
-    <origin xyz="0.150 0 0.300" rpy="0 3.14 3.14" />
-  </xacro:us_sensor-->
-  <!-- SENSOR 7 -->
-  <!-- xacro:us_sensor name="us_7" parent="base_link">
-    <origin xyz="0.160 0 0.300" rpy="0 3.14 3.14" />
-  </xacro:us_sensor-->
-  <!-- SENSOR 8 -->
-  <!-- xacro:us_sensor name="us_8" parent="base_link">
-    <origin xyz="0.170 0 0.300" rpy="0 3.14 3.14" />
-  </xacro:us_sensor-->
-  <!-- SENSOR 9 -->
-  <!-- xacro:us_sensor name="us_9" parent="base_link">
-    <origin xyz="0.180 0 0.300" rpy="0 3.14 3.14" />
-  </xacro:us_sensor-->
-  <!-- SENSOR 10 -->
-  <!-- xacro:us_sensor name="us_10" parent="base_link">
-    <origin xyz="0.100 0 0.300" rpy="0 3.14 3.14" />
-  </xacro:us_sensor-->
-  <!-- SENSOR 11 -->
-  <!-- xacro:us_sensor name="us_11" parent="base_link">
-    <origin xyz="0.100 0 0.300" rpy="0 3.14 3.14" />
-  </xacro:us_sensor-->
-  <!-- SENSOR 12 -->
-  <!-- xacro:us_sensor name="us_12" parent="base_link">
-    <origin xyz="0.190 0 0.300" rpy="0 3.14 3.14" />
-  </xacro:us_sensor-->
-  <!-- SENSOR 13 -->
-  <!-- xacro:us_sensor name="us_13" parent="base_link">
-    <origin xyz="0.200 0 0.300" rpy="0 3.14 3.14" />
-  </xacro:us_sensor-->
-  <!-- SENSOR 14 -->
-  <!-- xacro:us_sensor name="us_14" parent="base_link">
-    <origin xyz="0.210 0 0.300" rpy="0 3.14 3.14" />
-  </xacro:us_sensor-->
-  <!-- SENSOR 15 -->
-  <!-- xacro:us_sensor name="us_15" parent="base_link">
-    <origin xyz="0.220 0 0.300" rpy="0 3.14 3.14" />
-  </xacro:us_sensor-->
-  <!-- SENSOR 16 -->
-  <!-- xacro:us_sensor name="us_16" parent="base_link">
-    <origin xyz="0.230 0 0.300" rpy="0 3.14 3.14" />
-  </xacro:us_sensor-->
-  <!--Camera  -->
-  <!-- <xacro:camera name="camera" parent="base_link">
-    <origin xyz="0 0 0.38" rpy="0 0 0" />
-  </xacro:camera> -->
-  <!--cabinet-->
-  <!--   <xacro:mmo_500_cabinet name="cabinet" parent="base_link">
-  	<origin xyz="0.072 0 0.386" rpy="0 0 0" />
-  </xacro:mmo_500_cabinet>
- -->
-  <!--ur10-->
-  <!--  <xacro:ur10_robot parent="cabinet_link" prefix="ur10" joint_limited="true"
-		 shoulder_pan_lower_limit="${-pi}" shoulder_pan_upper_limit="${pi}"
-		 shoulder_lift_lower_limit="${-pi}" shoulder_lift_upper_limit="${pi}"
-		 elbow_joint_lower_limit="${-pi}" elbow_joint_upper_limit="${pi}"
-		 wrist_1_lower_limit="${-pi}" wrist_1_upper_limit="${pi}"
-		 wrist_2_lower_limit="${-pi}" wrist_2_upper_limit="${pi}"
-		 wrist_3_lower_limit="${-pi}" wrist_3_upper_limit="${pi}">
-  </xacro:ur10_robot> -->
-  <!--ur5-->
-  <!--   <xacro:ur5_robot parent="cabinet_link" prefix="ur5" joint_limited="true"
-     shoulder_pan_lower_limit="${-pi}" shoulder_pan_upper_limit="${pi}"
-     shoulder_lift_lower_limit="${-pi}" shoulder_lift_upper_limit="${pi}"
-     elbow_joint_lower_limit="${-pi}" elbow_joint_upper_limit="${pi}"
-     wrist_1_lower_limit="${-pi}" wrist_1_upper_limit="${pi}"
-     wrist_2_lower_limit="${-pi}" wrist_2_upper_limit="${pi}"
-     wrist_3_lower_limit="${-pi}" wrist_3_upper_limit="${pi}">
-  </xacro:ur5_robot> -->
-  <!-- Pilz arm -->
-  <!--     <xacro:prbt parent="cabinet_link" prefix="pilz">
-    <origin xyz="0 0 0." rpy="0 0 0" />
-  </xacro:prbt> -->
+  <!-- Realsense D435 -->
+  <xacro:if value="${d435 == True}">
+    <xacro:include filename="$(find realsense2_description)/urdf/_d435.urdf.xacro"/>
+    <xacro:sensor_d435 parent="base_link">
+      <origin xyz="0.292 0.0 0.716" rpy="0 0 0"/>
+    </xacro:sensor_d435>
+  </xacro:if>
+  <!-- Using IMU -->
+  <xacro:if value="${imu == True}">
+    <link name="imu_link">
+      <inertial>
+        <mass value="0.001" />
+        <origin xyz="0 0 0" rpy="0 0 0" />
+        <inertia ixx="0.0001" ixy="0" ixz="0" iyy="0.000001" iyz="0" izz="0.0001" />
+      </inertial>
+    </link>
+    <joint name="imu2_joint" type="fixed">
+      <axis xyz="0 1 0"/>
+      <origin rpy="0 0 0" xyz="-0.052 0.208 0.266"/>
+      <parent link="base_link"/>
+      <child link="imu_link"/>
+    </joint>
+  </xacro:if>
+  <!-- Universal arms -->
+  <xacro:unless value="${arm == ''}">
+    <xacro:arg name="tf_prefix" default="${arm}" />
+    <xacro:arg name="joint_limit_params" default="$(find ur_description)/config/$(arg arm_type)/joint_limits.yaml"/>
+    <xacro:arg name="kinematics_params" default="$(find ur_description)/config/$(arg arm_type)/default_kinematics.yaml"/>
+    <xacro:arg name="physical_params" default="$(find ur_description)/config/$(arg arm_type)/physical_parameters.yaml"/>
+    <xacro:arg name="visual_params" default="$(find ur_description)/config/$(arg arm_type)/visual_parameters.yaml"/>
+    <xacro:arg name="transmission_hw_interface" default=""/>
+    <xacro:arg name="safety_limits" default="false"/>
+    <xacro:arg name="safety_pos_margin" default="0.15"/>
+    <xacro:arg name="safety_k_position" default="20"/>
+    <xacro:arg name="force_abs_paths" default="false" />
+    <!-- cabinet link -->
+    <joint name="cabinet_joint" type="fixed">
+      <origin xyz="0.072 0 0.386" rpy="0 0 0" />
+      <joint_properties damping="1" friction="1"/>
+      <parent link="base_link"/>
+      <child link="cabinet_link"/>
+    </joint>
+    <link name="cabinet_link">
+      <inertial>
+        <mass value="2"/>
+        <origin rpy="0 0 -1.5708" xyz="0 0 0"/>
+        <inertia ixx="0.457072" ixy="0.0" ixz="0.0" iyy="0.23616" iyz="0.0" izz="0.686"/>
+      </inertial>
+      <visual>
+        <origin rpy="0 0 -1.5708" xyz="0 0 0"/>
+        <geometry>
+          <mesh filename="package://neo_mpo_700-2/robot_model/mpo_700/meshes/cabin.dae" scale="0.001 0.001 0.001"/>
+        </geometry>
+      </visual>
+      <collision>
+        <origin rpy="0 0 -1.5708" xyz="0. 0. 0"/>
+        <geometry>
+          <mesh filename="package://neo_mpo_700-2/robot_model/mpo_700/meshes/cabin.dae" scale="0.001 0.001 0.001"/>
+        </geometry>
+      </collision>
+    </link>
+    <!-- arm link -->
+    <xacro:include filename="$(find ur_description)/urdf/ur_macro.xacro"/>
+    <xacro:ur_robot name="${arm}"
+      parent="cabinet_link"
+      tf_prefix="$(arg tf_prefix)"
+      joint_limits_parameters_file="$(arg joint_limit_params)"
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
Commit message: fixing URDF path

File: robot_model/mpo_500/mpo_500.urdf.xacro (robot description, xacro)
@@ -18,5 +18,5 @@
   </xacro:unless>
   <link name="base_link"/>
-  <joint name="base_footprint_joint" type="${meca_joint_type}">
+  <joint name="base_footprint_joint" type="fixed">
     <origin rpy="0 0 0" xyz="0 0 0"/>
     <axis xyz="0 0 -1"/>
@@ -34,5 +34,5 @@
       <origin rpy="-1.571 0 1.571" xyz="0. 0. 0"/>
       <geometry>
-        <mesh filename="package://neo_mpo_500-2/robot_model/meshes/MPO_500/MPO-500-BODY.dae" scale="0.001 0.001 0.001"/>
+        <mesh filename="package://neo_mpo_500-2/robot_model/mpo_500/meshes/MPO-500-BODY.dae" scale="0.001 0.001 0.001"/>
       </geometry>
     </visual>
@@ -40,5 +40,5 @@
       <origin rpy="-1.571 0 1.571" xyz="0. 0. 0.0"/>
       <geometry>
-        <mesh filename="package://neo_mpo_500-2/robot_model/meshes/MPO_500/MPO-500-BODY.dae" scale="0.001 0.001 0.001"/>
+        <mesh filename="package://neo_mpo_500-2/robot_model/mpo_500/meshes/MPO-500-BODY.dae" scale="0.001 0.001 0.001"/>
       </geometry>
     </collision>
@@ -62,11 +62,11 @@
       <origin rpy="0 0 0" xyz="0 0 0"/>
       <geometry>
-        <mesh filename="package://neo_mpo_500-2/robot_model/meshes/MPO_500/MPO-500-WHEEL.dae" scale="0.001 0.001 0.001"/>
-      </geometry>
-    </visual>
-    <collision>
-      <origin rpy="0 0 0" xyz="0 0 0"/>
-      <geometry>
-        <mesh filename="package://neo_mpo_500-2/robot_model/meshes/MPO_500/MPO-500-WHEEL.dae" scale="0.001 0.001 0.001"/>
+        <mesh filename="package://neo_mpo_500-2/robot_model/mpo_500/meshes/MPO-500-WHEEL.dae" scale="0.001 0.001 0.001"/>
+      </geometry>
+    </visual>
+    <collision>
+      <origin rpy="0 0 0" xyz="0 0 0"/>
+      <geometry>
+        <mesh filename="package://neo_mpo_500-2/robot_model/mpo_500/meshes/MPO-500-WHEEL.dae" scale="0.001 0.001 0.001"/>
       </geometry>
     </collision>
@@ -90,11 +90,11 @@
       <origin rpy="0 0 0" xyz="0 0 0"/>
       <geometry>
-        <mesh filename="package://neo_mpo_500-2/robot_model/meshes/MPO_500/MPO-500-WHEEL.dae" scale="0.001 0.001 0.001"/>
-      </geometry>
-    </visual>
-    <collision>
-      <origin rpy="0 0 0" xyz="0 0 0"/>
-      <geometry>
-        <mesh filename="package://neo_mpo_500-2/robot_model/meshes/MPO_500/MPO-500-WHEEL.dae" scale="0.001 0.001 0.001"/>
+        <mesh filename="package://neo_mpo_500-2/robot_model/mpo_500/meshes/MPO-500-WHEEL.dae" scale="0.001 0.001 0.001"/>
+      </geometry>
+    </visual>
+    <collision>
+      <origin rpy="0 0 0" xyz="0 0 0"/>
+      <geometry>
+        <mesh filename="package://neo_mpo_500-2/robot_model/mpo_500/meshes/MPO-500-WHEEL.dae" scale="0.001 0.001 0.001"/>
       </geometry>
     </collision>
@@ -118,11 +118,11 @@
       <origin rpy="0 0 0" xyz="0 0 0"/>
       <geometry>
-        <mesh filename="package://neo_mpo_500-2/robot_model/meshes/MPO_500/MPO-500-WHEEL.dae" scale="0.001 0.001 0.001"/>
-      </geometry>
-    </visual>
-    <collision>
-      <origin rpy="0 0 0" xyz="0 0 0"/>
-      <geometry>
-        <mesh filename="package://neo_mpo_500-2/robot_model/meshes/MPO_500/MPO-500-WHEEL.dae" scale="0.001 0.001 0.001"/>
+        <mesh filename="package://neo_mpo_500-2/robot_model/mpo_500/meshes/MPO-500-WHEEL.dae" scale="0.001 0.001 0.001"/>
+      </geometry>
+    </visual>
+    <collision>
+      <origin rpy="0 0 0" xyz="0 0 0"/>
+      <geometry>
+        <mesh filename="package://neo_mpo_500-2/robot_model/mpo_500/meshes/MPO-500-WHEEL.dae" scale="0.001 0.001 0.001"/>
       </geometry>
     </collision>
@@ -146,11 +146,11 @@
       <origin rpy="0 0 0" xyz="0 0 0"/>
       <geometry>
-        <mesh filename="package://neo_mpo_500-2/robot_model/meshes/MPO_500/MPO-500-WHEEL.dae" scale="0.001 0.001 0.001"/>
-      </geometry>
-    </visual>
-    <collision>
-      <origin rpy="0 0 0" xyz="0 0 0"/>
-      <geometry>
-        <mesh filename="package://neo_mpo_500-2/robot_model/meshes/MPO_500/MPO-500-WHEEL.dae" scale="0.001 0.001 0.001"/>
+        <mesh filename="package://neo_mpo_500-2/robot_model/mpo_500/meshes/MPO-500-WHEEL.dae" scale="0.001 0.001 0.001"/>
+      </geometry>
+    </visual>
+    <collision>
+      <origin rpy="0 0 0" xyz="0 0 0"/>
+      <geometry>
+        <mesh filename="package://neo_mpo_500-2/robot_model/mpo_500/meshes/MPO-500-WHEEL.dae" scale="0.001 0.001 0.001"/>
       </geometry>
     </collision>
@@ -171,11 +171,11 @@
       <origin rpy="-1.57 0 3.14" xyz="0 0 -0.12"/>
       <geometry>
-        <mesh filename="package://neo_mpo_500-2/robot_model/meshes/MPO_500/SICK-S300.dae" scale="0.001 0.001 0.001"/>
-      </geometry>
-    </visual>
-    <collision>
-      <origin rpy="-1.57 0 3.14" xyz="0 0 -0.12"/>
-      <geometry>
-        <mesh filename="package://neo_mpo_500-2/robot_model/meshes/MPO_500/SICK-S300.dae" scale="0.001 0.001 0.001"/>
+        <mesh filename="package://neo_mpo_500-2/robot_model/mpo_500/meshes/SICK-S300.dae" scale="0.001 0.001 0.001"/>
+      </geometry>
+    </visual>
+    <collision>
+      <origin rpy="-1.57 0 3.14" xyz="0 0 -0.12"/>
+      <geometry>
+        <mesh filename="package://neo_mpo_500-2/robot_model/mpo_500/meshes/SICK-S300.dae" scale="0.001 0.001 0.001"/>
       </geometry>
     </collision>
@@ -196,11 +196,11 @@
       <origin rpy="-1.57 0 3.14" xyz="0 0 -0.12"/>
       <geometry>
-        <mesh filename="package://neo_mpo_500-2/robot_model/meshes/MPO_500/SICK-S300.dae" scale="0.001 0.001 0.001"/>
-      </geometry>
-    </visual>
-    <collision>
-      <origin rpy="-1.57 0 3.14" xyz="0 0 -0.12"/>
-      <geometry>
-        <mesh filename="package://neo_mpo_500-2/robot_model/meshes/MPO_500/SICK-S300.dae" scale="0.001 0.001 0.001"/>
+        <mesh filename="package://neo_mpo_500-2/robot_model/mpo_500/meshes/SICK-S300.dae" scale="0.001 0.001 0.001"/>
+      </geometry>
+    </visual>
+    <collision>
+      <origin rpy="-1.57 0 3.14" xyz="0 0 -0.12"/>
+      <geometry>
+        <mesh filename="package://neo_mpo_500-2/robot_model/mpo_500/meshes/SICK-S300.dae" scale="0.001 0.001 0.001"/>
       </geometry>
     </collision>
