Commit message: adjusting the visualization

File: robot_model/xacros/mpo_500_body.urdf.xacro (robot description, xacro)
@@ -47,5 +47,5 @@
       wheel_joint_type="${meca_joint_type}"
       >
-      <origin rpy="0 0 0" xyz="0.25 0.28 0.13"/>
+      <origin rpy="0 0 0" xyz="0.25 0.274 0.127"/>
     </xacro:mpo_500_omni_wheel>
     <xacro:mpo_500_omni_wheel
@@ -54,5 +54,5 @@
       wheel_joint_type="${meca_joint_type}"
       >
-      <origin rpy="0 0 3.14" xyz="0.25 -0.28 0.13"/>
+      <origin rpy="0 0 3.14" xyz="0.25 -0.274 0.127"/>
     </xacro:mpo_500_omni_wheel>
     <xacro:mpo_500_omni_wheel
@@ -61,5 +61,5 @@
       wheel_joint_type="${meca_joint_type}"
       >
-      <origin rpy="0 0 0" xyz="-0.25 0.28 0.13"/>
+      <origin rpy="0 0 0" xyz="-0.25 0.274 0.127"/>
     </xacro:mpo_500_omni_wheel>
     <xacro:mpo_500_omni_wheel
@@ -68,5 +68,5 @@
       wheel_joint_type="${meca_joint_type}"
       >
-      <origin rpy="0 0 3.14" xyz="-0.25 -0.28 0.13"/>
+      <origin rpy="0 0 3.14" xyz="-0.25 -0.274 0.127"/>
     </xacro:mpo_500_omni_wheel>
   </xacro:macro>
